Commit message: Update my_robot.xacro

File: src/my_robot/urdf/my_robot.xacro (robot description, xacro)
@@ -54,3 +54,65 @@
     </visual>
   </link>
+  <link name='right_wheel'>
+    <collision name='collision'>
+      <origin xyz="0 0 0" rpy=" 0 1.5707 1.5707"/>
+      <geometry>
+        <cylinder size="0.1 0.05"/>
+      </geometry>
+    </collision>
+    <inertial>
+      <mass value="5.0"/>
+      <origin xyz="0 0 0" rpy=" 0 1.5707 1.5707"/>
+      <inertia
+          ixx="0.1" ixy="0" ixz="0"
+          iyy="0.1" iyz="0"
+          izz="0.1"
+      />
+    </inertial>
+    <visual name='chassis_visual'>
+      <origin xyz="0 0 0" rpy=" 0 1.5707 1.5707"/>
+      <geometry>
+        <cylinder size="0.1 0.05"/>
+      </geometry>
+    </visual>
+	<joint type="continuous" name="right_wheel_hinge">
+		<origin xyz="0 -0.15 0" rpy="0 0 0"/>
+		<child link="right_wheel"/>
+		<parent link="chassis"/>
+		<axis xyz="0 1 0" rpy="0 0 0"/>
+		<limit effort="10000" velocity="1000"/>
+		<dynamics damping="1.0" friction="1.0"/>
+	</joint>
+  </link>
+  <link name='left_wheel'>
+    <collision name='collision'>
+      <origin xyz="0 0 0" rpy=" 0 1.5707 1.5707"/>
+      <geometry>
+        <cylinder size="0.1 0.05"/>
+      </geometry>
+    </collision>
+    <inertial>
+      <mass value="5.0"/>
+      <origin xyz="0 0 0" rpy=" 0 1.5707 1.5707"/>
+      <inertia
+          ixx="0.1" ixy="0" ixz="0"
+          iyy="0.1" iyz="0"
+          izz="0.1"
+      />
+    </inertial>
+    <visual name='chassis_visual'>
+      <origin xyz="0 0 0" rpy=" 0 1.5707 1.5707"/>
+      <geometry>
+        <cylinder size="0.1 0.05"/>
+      </geometry>
+    </visual>
+	<joint type="continuous" name="left_wheel_hinge">
+		<origin xyz="0 0.15 0" rpy="0 0 0"/>
+		<child link="left_wheel"/>
+		<parent link="chassis"/>
+		<axis xyz="0 1 0" rpy="0 0 0"/>
+		<limit effort="10000" velocity="1000"/>
+		<dynamics damping="1.0" friction="1.0"/>
+	</joint>
+  </link>
 </robot>

Commit message: Update my_robot.xacro

File: src/my_robot/urdf/my_robot.xacro (robot description, xacro)
@@ -1,3 +1,4 @@
 <robot name="my_robot" xmlns:xacro="http://www.ros.org/wiki/xacro">
+  <xacro:include filename="$(find my_robot)/urdf/my_robot.gazebo" />
   <link name="robot_footprint"></link>
   <joint name="robot_footprint_joint" type="fixed">
@@ -55,8 +56,9 @@
   </link>
   <link name='right_wheel'>
+   <pose>0 0 0 0 0 0</pose>
     <collision name='collision'>
       <origin xyz="0 0 0" rpy=" 0 1.5707 1.5707"/>
       <geometry>
-        <cylinder size="0.1 0.05"/>
+        <cylinder length="0.05" radius="0.1"/>
       </geometry>
     </collision>
@@ -70,10 +72,11 @@
       />
     </inertial>
-    <visual name='chassis_visual'>
+    <visual name='visual'>
       <origin xyz="0 0 0" rpy=" 0 1.5707 1.5707"/>
       <geometry>
-        <cylinder size="0.1 0.05"/>
+        <cylinder length="0.05" radius="0.1"/>
       </geometry>
     </visual>
+</link>
 	<joint type="continuous" name="right_wheel_hinge">
 		<origin xyz="0 -0.15 0" rpy="0 0 0"/>
@@ -84,10 +87,10 @@
 		<dynamics damping="1.0" friction="1.0"/>
 	</joint>
-  </link>
   <link name='left_wheel'>
+   <pose>0 0 0 0 0 0</pose>
     <collision name='collision'>
       <origin xyz="0 0 0" rpy=" 0 1.5707 1.5707"/>
       <geometry>
-        <cylinder size="0.1 0.05"/>
+        <cylinder length="0.05" radius="0.1"/>
       </geometry>
     </collision>
@@ -101,10 +104,11 @@
       />
     </inertial>
-    <visual name='chassis_visual'>
+    <visual name='visual'>
       <origin xyz="0 0 0" rpy=" 0 1.5707 1.5707"/>
       <geometry>
-        <cylinder size="0.1 0.05"/>
+        <cylinder length="0.05" radius="0.1"/>
       </geometry>
     </visual>
+  </link>
 	<joint type="continuous" name="left_wheel_hinge">
 		<origin xyz="0 0.15 0" rpy="0 0 0"/>
@@ -115,4 +119,63 @@
 		<dynamics damping="1.0" friction="1.0"/>
 	</joint>
+  <link name="camera">
+	<pose>0 0 0 0 0 0</pose>
+    <inertial>
+      <mass value="0.1"/>
+      <origin xyz="0.0 0 0" rpy=" 0 0 0"/>
+      <inertia
+          ixx="1e-6" ixy="0" ixz="0"
+          iyy="1e-6" iyz="0"
+          izz="1e-6"
+      />
+    </inertial>
+    <collision name='collision'>
+      <origin xyz="0 0 0" rpy=" 0 0 0"/>
+      <geometry>
+        <box size="0.05, 0.05, 0.05"/>
+      </geometry>
+    </collision>
+    <visual name='visual'>
+      <origin xyz="0 0 0" rpy=" 0 0 0"/>
+      <geometry>
+        <box size="0.05, 0.05, 0.05"/>
+      </geometry>
+    </visual>
   </link>
+  <joint name="camera_joint" type="fixed">
+    <origin xyz="0.2 0 0" rpy="0 0 0" />
+    <parent link="chassis"/>
+    <child link="camera" />
+    <axis xyz="0 1 0" rpy="0 0 0"/>
+  </joint>
+  <link name="hokuyo">
+      <pose>0 0 0 0 0 0</pose>
+    <inertial>
+      <mass value="1e-5"/>
+      <origin xyz="0 0 0" rpy=" 0 0 0"/>
+      <inertia
+          ixx="1e-6" ixy="0" ixz="0"
+          iyy="1e-6" iyz="0"
+          izz="1e-6"
+      />
+    </inertial>
+    <collision name='collision'>
+      <origin xyz="0 0 0" rpy=" 0 0 0"/>
+      <geometry>
+        <box size="0.1, 0.1, 0.1"/>
+      </geometry>
+    </collision>
+    <visual name='visual'>
+      <origin xyz="0 0 0" rpy=" 0 0 0"/>
+      <geometry>
+        <mesh filename="package://my_robot/meshes/hokuyo.dae"/>
+      </geometry>
+    </visual>
+  </link>
+ <joint name="hokuyo_joint" type="fixed">
+    <origin xyz="0.15 0 0.1" rpy="0 0 0" />
+    <parent link="chassis"/>
+    <child link="hokuyo" />
+    <axis xyz="0 1 0" rpy="0 0 0"/>
+  </joint>
 </robot>

Commit message: Update my_robot.xacro

File: src/my_robot/urdf/my_robot.xacro (robot description, xacro)
@@ -1,2 +1,3 @@
+<?xml version='1.0'?>
 <robot name="my_robot" xmlns:xacro="http://www.ros.org/wiki/xacro">
   <xacro:include filename="$(find my_robot)/urdf/my_robot.gazebo" />
@@ -55,4 +56,5 @@
     </visual>
   </link>
+<!-- Add two wheels -->
   <link name='right_wheel'>
    <pose>0 0 0 0 0 0</pose>
@@ -119,17 +121,15 @@
 		<dynamics damping="1.0" friction="1.0"/>
 	</joint>
+  <!-- Add camera -->
   <link name="camera">
-	<pose>0 0 0 0 0 0</pose>
+	<origin xyz="0 0 0" rpy="0 0 0" />
     <inertial>
       <mass value="0.1"/>
-      <origin xyz="0.0 0 0" rpy=" 0 0 0"/>
       <inertia
           ixx="1e-6" ixy="0" ixz="0"
-          iyy="1e-6" iyz="0"
-          izz="1e-6"
+          iyy="1e-6" iyz="0" izz="1e-6"
       />
     </inertial>
     <collision name='collision'>
-      <origin xyz="0 0 0" rpy=" 0 0 0"/>
       <geometry>
         <box size="0.05, 0.05, 0.05"/>
@@ -137,5 +137,4 @@
     </collision>
     <visual name='visual'>
-      <origin xyz="0 0 0" rpy=" 0 0 0"/>
       <geometry>
         <box size="0.05, 0.05, 0.05"/>
@@ -144,22 +143,20 @@
   </link>
   <joint name="camera_joint" type="fixed">
+    <axis xyz="0 1 0"/>
     <origin xyz="0.2 0 0" rpy="0 0 0" />
     <parent link="chassis"/>
     <child link="camera" />
-    <axis xyz="0 1 0" rpy="0 0 0"/>
   </joint>
+  <!-- Add Lidar -->
   <link name="hokuyo">
-      <pose>0 0 0 0 0 0</pose>
+    <origin xyz="0 0 0" rpy="0 0 0" />
     <inertial>
       <mass value="1e-5"/>
-      <origin xyz="0 0 0" rpy=" 0 0 0"/>
       <inertia
           ixx="1e-6" ixy="0" ixz="0"
-          iyy="1e-6" iyz="0"
-          izz="1e-6"
+          iyy="1e-6" iyz="0" izz="1e-6"
       />
     </inertial>
     <collision name='collision'>
-      <origin xyz="0 0 0" rpy=" 0 0 0"/>
       <geometry>
         <box size="0.1, 0.1, 0.1"/>
@@ -167,5 +164,4 @@
     </collision>
     <visual name='visual'>
-      <origin xyz="0 0 0" rpy=" 0 0 0"/>
       <geometry>
         <mesh filename="package://my_robot/meshes/hokuyo.dae"/>
@@ -174,8 +170,8 @@
   </link>
  <joint name="hokuyo_joint" type="fixed">
+    <axis xyz="0 1 0" rpy="0 0 0"/>
     <origin xyz="0.15 0 0.1" rpy="0 0 0" />
     <parent link="chassis"/>
     <child link="hokuyo" />
-    <axis xyz="0 1 0" rpy="0 0 0"/>
   </joint>
 </robot>
