Commit message: Update my_robot.xacro

File: my_robot/urdf/my_robot.xacro (robot description, xacro)
@@ -19,5 +19,5 @@
       />
     </inertial>
-    <collision name='collision'>
+    <collision name='chassis_collision'>
       <origin xyz="0 0 0" rpy=" 0 0 0"/>
       <geometry>
@@ -59,5 +59,5 @@
   <link name='right_wheel'>
    <pose>0 0 0 0 0 0</pose>
-    <collision name='collision'>
+    <collision name='right_wheel_collision'>
       <origin xyz="0 0 0" rpy=" 0 1.5707 1.5707"/>
       <geometry>
@@ -74,5 +74,5 @@
       />
     </inertial>
-    <visual name='visual'>
+    <visual name='right_wheel_visual'>
       <origin xyz="0 0 0" rpy=" 0 1.5707 1.5707"/>
       <geometry>
@@ -91,5 +91,5 @@
   <link name='left_wheel'>
    <pose>0 0 0 0 0 0</pose>
-    <collision name='collision'>
+    <collision name='left_wheel_collision'>
       <origin xyz="0 0 0" rpy=" 0 1.5707 1.5707"/>
       <geometry>
@@ -106,5 +106,5 @@
       />
     </inertial>
-    <visual name='visual'>
+    <visual name='left_wheel_visual'>
       <origin xyz="0 0 0" rpy=" 0 1.5707 1.5707"/>
       <geometry>
@@ -131,12 +131,12 @@
       />
     </inertial>
-    <collision name='collision'>
+    <collision name='camera_collision'>
       <geometry>
-        <box size="0.05, 0.05, 0.05"/>
+        <box size="0.05 0.05 0.05"/>
       </geometry>
     </collision>
-    <visual name='visual'>
+    <visual name='camera_visual'>
       <geometry>
-        <box size="0.05, 0.05, 0.05"/>
+        <box size="0.05 0.05 0.05"/>
       </geometry>
     </visual>
@@ -158,10 +158,10 @@
       />
     </inertial>
-    <collision name='collision'>
+    <collision name='hokuyo_collision'>
       <geometry>
-        <box size="0.1, 0.1, 0.1"/>
+        <box size="0.1 0.1 0.1"/>
       </geometry>
     </collision>
-    <visual name='visual'>
+    <visual name='hokuyo_visual'>
       <geometry>
         <mesh filename="package://my_robot/meshes/hokuyo.dae"/>

Commit message: Update my_robot.xacro

File: my_robot/urdf/my_robot.xacro (robot description, xacro)
@@ -175,3 +175,15 @@
     <child link="hokuyo" />
   </joint>
+<gazebo reference="left_wheel">
+    <material>Gazebo/Red</material>
+</gazebo>
+<gazebo reference="right_wheel">
+    <material>Gazebo/Red</material>
+</gazebo>
+<gazebo reference="chassis">
+    <material>Gazebo/Yellow</material>
+</gazebo>
+<gazebo reference="camera">
+    <material>Gazebo/Blue</material>
+</gazebo>
 </robot>

Commit message: Update my_robot.xacro

File: my_robot/urdf/my_robot.xacro (robot description, xacro)
@@ -22,5 +22,5 @@
       <origin xyz="0 0 0" rpy=" 0 0 0"/>
       <geometry>
-        <box size=".4 .2 .1"/>
+        <box size=".4 .4 .1"/>
       </geometry>
     </collision>
@@ -28,5 +28,5 @@
       <origin xyz="0 0 0" rpy=" 0 0 0"/>
       <geometry>
-        <box size=".4 .2 .1"/>
+        <box size=".4 .4 .1"/>
       </geometry>
     </visual>
@@ -34,5 +34,5 @@
       <origin xyz="-0.15 0 -0.05" rpy=" 0 0 0"/>
       <geometry>
-        <sphere radius="0.0499"/>
+        <sphere radius="0.075"/>
       </geometry>
     </collision>
@@ -40,5 +40,5 @@
       <origin xyz="-0.15 0 -0.05" rpy=" 0 0 0"/>
       <geometry>
-        <sphere radius="0.05"/>
+        <sphere radius="0.075"/>
       </geometry>
     </visual>
@@ -46,5 +46,5 @@
       <origin xyz="0.15 0 -0.05" rpy=" 0 0 0"/>
       <geometry>
-        <sphere radius="0.0499"/>
+        <sphere radius="0.075"/>
       </geometry>
     </collision>
@@ -52,5 +52,5 @@
       <origin xyz="0.15 0 -0.05" rpy=" 0 0 0"/>
       <geometry>
-        <sphere radius="0.05"/>
+        <sphere radius="0.075"/>
       </geometry>
     </visual>
@@ -62,5 +62,5 @@
       <origin xyz="0 0 0" rpy=" 0 1.5707 1.5707"/>
       <geometry>
-        <cylinder length="0.05" radius="0.1"/>
+        <cylinder length="0.075" radius="0.1"/>
       </geometry>
     </collision>
@@ -77,5 +77,5 @@
       <origin xyz="0 0 0" rpy=" 0 1.5707 1.5707"/>
       <geometry>
-        <cylinder length="0.05" radius="0.1"/>
+        <cylinder length="0.075" radius="0.1"/>
       </geometry>
     </visual>
@@ -94,5 +94,5 @@
       <origin xyz="0 0 0" rpy=" 0 1.5707 1.5707"/>
       <geometry>
-        <cylinder length="0.05" radius="0.1"/>
+        <cylinder length="0.075" radius="0.1"/>
       </geometry>
     </collision>
@@ -109,5 +109,5 @@
       <origin xyz="0 0 0" rpy=" 0 1.5707 1.5707"/>
       <geometry>
-        <cylinder length="0.05" radius="0.1"/>
+        <cylinder length="0.075" radius="0.1"/>
       </geometry>
     </visual>

Commit message: Update my_robot.xacro

File: my_robot/urdf/my_robot.xacro (robot description, xacro)
@@ -22,5 +22,5 @@
       <origin xyz="0 0 0" rpy=" 0 0 0"/>
       <geometry>
-        <box size=".4 .4 .1"/>
+        <box size=".4 .3 .1"/>
       </geometry>
     </collision>
@@ -28,5 +28,5 @@
       <origin xyz="0 0 0" rpy=" 0 0 0"/>
       <geometry>
-        <box size=".4 .4 .1"/>
+        <box size=".4 .3 .1"/>
       </geometry>
     </visual>
@@ -34,5 +34,5 @@
       <origin xyz="-0.15 0 -0.05" rpy=" 0 0 0"/>
       <geometry>
-        <sphere radius="0.075"/>
+        <sphere radius="0.06"/>
       </geometry>
     </collision>
@@ -40,5 +40,5 @@
       <origin xyz="-0.15 0 -0.05" rpy=" 0 0 0"/>
       <geometry>
-        <sphere radius="0.075"/>
+        <sphere radius="0.06"/>
       </geometry>
     </visual>
@@ -46,5 +46,5 @@
       <origin xyz="0.15 0 -0.05" rpy=" 0 0 0"/>
       <geometry>
-        <sphere radius="0.075"/>
+        <sphere radius="0.06"/>
       </geometry>
     </collision>
@@ -52,5 +52,5 @@
       <origin xyz="0.15 0 -0.05" rpy=" 0 0 0"/>
       <geometry>
-        <sphere radius="0.075"/>
+        <sphere radius="0.06"/>
       </geometry>
     </visual>
@@ -82,5 +82,5 @@
 </link>
 	<joint type="continuous" name="right_wheel_hinge">
-		<origin xyz="0 -0.15 0" rpy="0 0 0"/>
+		<origin xyz="0 -0.2 0" rpy="0 0 0"/>
 		<child link="right_wheel"/>
 		<parent link="chassis"/>
@@ -114,5 +114,5 @@
   </link>
 	<joint type="continuous" name="left_wheel_hinge">
-		<origin xyz="0 0.15 0" rpy="0 0 0"/>
+		<origin xyz="0 0.2 0" rpy="0 0 0"/>
 		<child link="left_wheel"/>
 		<parent link="chassis"/>

Commit message: Update my_robot.xacro

File: my_robot/urdf/my_robot.xacro (robot description, xacro)
@@ -34,5 +34,5 @@
       <origin xyz="-0.15 0 -0.05" rpy=" 0 0 0"/>
       <geometry>
-        <sphere radius="0.06"/>
+        <sphere radius="0.05"/>
       </geometry>
     </collision>
@@ -40,5 +40,5 @@
       <origin xyz="-0.15 0 -0.05" rpy=" 0 0 0"/>
       <geometry>
-        <sphere radius="0.06"/>
+        <sphere radius="0.05"/>
       </geometry>
     </visual>
@@ -46,5 +46,5 @@
       <origin xyz="0.15 0 -0.05" rpy=" 0 0 0"/>
       <geometry>
-        <sphere radius="0.06"/>
+        <sphere radius="0.05"/>
       </geometry>
     </collision>
@@ -52,5 +52,5 @@
       <origin xyz="0.15 0 -0.05" rpy=" 0 0 0"/>
       <geometry>
-        <sphere radius="0.06"/>
+        <sphere radius="0.05"/>
       </geometry>
     </visual>

Commit message: Update my_robot.xacro

File: my_robot/urdf/my_robot.xacro (robot description, xacro)
@@ -11,5 +11,5 @@
     <pose>0 0 0.1 0 0 0</pose>
     <inertial>
-      <mass value="15.0"/>
+      <mass value="25.0"/>
       <origin xyz="0.0 0 0" rpy=" 0 0 0"/>
       <inertia
@@ -22,5 +22,5 @@
       <origin xyz="0 0 0" rpy=" 0 0 0"/>
       <geometry>
-        <box size=".4 .3 .1"/>
+        <box size=".8 .4 .2"/>
       </geometry>
     </collision>
@@ -28,29 +28,29 @@
       <origin xyz="0 0 0" rpy=" 0 0 0"/>
       <geometry>
-        <box size=".4 .3 .1"/>
+        <box size=".8 .4 .2"/>
       </geometry>
     </visual>
     <collision name='back_caster_collision'>
-      <origin xyz="-0.15 0 -0.05" rpy=" 0 0 0"/>
+      <origin xyz="-0.25 0 -0.1" rpy=" 0 0 0"/>
       <geometry>
-        <sphere radius="0.05"/>
+        <sphere radius="0.099"/>
       </geometry>
     </collision>
     <visual name='back_caster_visual'>
-      <origin xyz="-0.15 0 -0.05" rpy=" 0 0 0"/>
+      <origin xyz="-0.25 0 -0.1" rpy=" 0 0 0"/>
       <geometry>
-        <sphere radius="0.05"/>
+        <sphere radius="0.099"/>
       </geometry>
     </visual>
     <collision name='front_caster_collision'>
-      <origin xyz="0.15 0 -0.05" rpy=" 0 0 0"/>
+      <origin xyz="-0.25 0 -0.1" rpy=" 0 0 0"/>
       <geometry>
-        <sphere radius="0.05"/>
+        <sphere radius="0.099"/>
       </geometry>
     </collision>
     <visual name='front_caster_visual'>
-      <origin xyz="0.15 0 -0.05" rpy=" 0 0 0"/>
+      <origin xyz="-0.25 0 -0.1" rpy=" 0 0 0"/>
       <geometry>
-        <sphere radius="0.05"/>
+        <sphere radius="0.099"/>
       </geometry>
     </visual>
@@ -58,14 +58,8 @@
 <!-- Add two wheels -->
   <link name='right_wheel'>
-   <pose>0 0 0 0 0 0</pose>
-    <collision name='right_wheel_collision'>
-      <origin xyz="0 0 0" rpy=" 0 1.5707 1.5707"/>
-      <geometry>
-        <cylinder length="0.075" radius="0.1"/>
-      </geometry>
-    </collision>
+   <pose>0 0 0.8 0 0 0</pose>
     <inertial>
       <mass value="5.0"/>
-      <origin xyz="0 0 0" rpy=" 0 1.5707 1.5707"/>
+      <origin xyz="0 0 0" rpy=" 0 0 0"/>
       <inertia
           ixx="0.1" ixy="0" ixz="0"
@@ -74,13 +68,19 @@
       />
     </inertial>
+    <collision name='right_wheel_collision'>
+      <origin xyz="0 0 0" rpy=" 0 1.5707 1.5707"/>
+      <geometry>
+        <cylinder length="0.2" radius="0.05"/>
+      </geometry>
+    </collision>
     <visual name='right_wheel_visual'>
       <origin xyz="0 0 0" rpy=" 0 1.5707 1.5707"/>
       <geometry>
-        <cylinder length="0.075" radius="0.1"/>
+        <cylinder length="0.2" radius="0.05"/>
       </geometry>
     </visual>
 </link>
 	<joint type="continuous" name="right_wheel_hinge">
-		<origin xyz="0 -0.2 0" rpy="0 0 0"/>
+		<origin xyz="0 -0.3 0" rpy="0 0 0"/>
 		<child link="right_wheel"/>
 		<parent link="chassis"/>
@@ -90,14 +90,8 @@
 	</joint>
   <link name='left_wheel'>
-   <pose>0 0 0 0 0 0</pose>
-    <collision name='left_wheel_collision'>
-      <origin xyz="0 0 0" rpy=" 0 1.5707 1.5707"/>
-      <geometry>
-        <cylinder length="0.075" radius="0.1"/>
-      </geometry>
-    </collision>
+   <pose>0 0 0.8 0 0 0</pose>
     <inertial>
       <mass value="5.0"/>
-      <origin xyz="0 0 0" rpy=" 0 1.5707 1.5707"/>
+      <origin xyz="0 0 0" rpy=" 0 0 0"/>
       <inertia
           ixx="0.1" ixy="0" ixz="0"
@@ -106,13 +100,19 @@
       />
     </inertial>
+    <collision name='left_wheel_collision'>
+      <origin xyz="0 0 0" rpy=" 0 1.5707 1.5707"/>
+      <geometry>
+        <cylinder length="0.2" radius="0.05"/>
+      </geometry>
+    </collision>
     <visual name='left_wheel_visual'>
       <origin xyz="0 0 0" rpy=" 0 1.5707 1.5707"/>
       <geometry>
-        <cylinder length="0.075" radius="0.1"/>
+        <cylinder length="0.2" radius="0.05"/>
       </geometry>
     </visual>
   </link>
 	<joint type="continuous" name="left_wheel_hinge">
-		<origin xyz="0 0.2 0" rpy="0 0 0"/>
+		<origin xyz="0 0.3 0" rpy="0 0 0"/>
 		<child link="left_wheel"/>
 		<parent link="chassis"/>
@@ -122,46 +122,55 @@
 	</joint>
   <!-- Add camera -->
-  <link name="camera">
-	<origin xyz="0 0 0" rpy="0 0 0" />
+  <link name='camera'>
+    <pose>0 0 0 0 0 0</pose>
     <inertial>
       <mass value="0.1"/>
+      <origin xyz="0.0 0 0" rpy=" 0 0 0"/>
+      <box_inertia m="0.1" x="0.05" y="0.05" z="0.05"/>
       <inertia
           ixx="1e-6" ixy="0" ixz="0"
-          iyy="1e-6" iyz="0" izz="1e-6"
+          iyy="1e-6" iyz="0"
+          izz="1e-6"
       />
     </inertial>
-    <collision name='camera_collision'>
+    <collision name='collision'>
+      <origin xyz="0 0 0" rpy=" 0 0 0"/>
       <geometry>
-        <box size="0.05 0.05 0.05"/>
+        <box size=".05 .05 .05"/>
       </geometry>
     </collision>
     <visual name='camera_visual'>
+      <origin xyz="0 0 0" rpy=" 0 0 0"/>
       <geometry>
-        <box size="0.05 0.05 0.05"/>
+        <box size=".05 .05 .05"/>
       </geometry>
     </visual>
   </link>
-  <joint name="camera_joint" type="fixed">
-    <axis xyz="0 1 0"/>
-    <origin xyz="0.2 0 0" rpy="0 0 0" />
+  <joint type="fixed" name="camera_joint">
+    <origin xyz="0.4 0 0" rpy="0 0 0"/>
+    <child link="camera"/>
     <parent link="chassis"/>
-    <child link="camera" />
+    <axis xyz="0 1 0" rpy="0 0 0"/>
   </joint>
   <!-- Add Lidar -->
-  <link name="hokuyo">
-    <origin xyz="0 0 0" rpy="0 0 0" />
+  <link name='hokuyo'>
+    <pose>0 0 0 0 0 0</pose>
     <inertial>
       <mass value="1e-5"/>
+      <origin xyz="0.0 0 0" rpy=" 0 0 0"/>
       <inertia
           ixx="1e-6" ixy="0" ixz="0"
-          iyy="1e-6" iyz="0" izz="1e-6"
+          iyy="1e-6" iyz="0"
+          izz="1e-6"
       />
     </inertial>
-    <collision name='hokuyo_collision'>
+    <collision name='collision'>
+      <origin xyz="0 0 0" rpy=" 0 0 0"/>
       <geometry>
-        <box size="0.1 0.1 0.1"/>
+        <box size=".01 .01 .01"/>
       </geometry>
     </collision>
     <visual name='hokuyo_visual'>
+      <origin xyz="0 0 0" rpy=" 0 0 0"/>
       <geometry>
         <mesh filename="package://my_robot/meshes/hokuyo.dae"/>

Commit message: Update my_robot.xacro

File: my_robot/urdf/my_robot.xacro (robot description, xacro)
@@ -11,5 +11,5 @@
     <pose>0 0 0.1 0 0 0</pose>
     <inertial>
-      <mass value="25.0"/>
+      <mass value="30.0"/>
       <origin xyz="0.0 0 0" rpy=" 0 0 0"/>
       <inertia
@@ -34,5 +34,5 @@
       <origin xyz="-0.25 0 -0.1" rpy=" 0 0 0"/>
       <geometry>
-        <sphere radius="0.099"/>
+        <sphere radius="0.0998"/>
       </geometry>
     </collision>
@@ -40,5 +40,5 @@
       <origin xyz="-0.25 0 -0.1" rpy=" 0 0 0"/>
       <geometry>
-        <sphere radius="0.099"/>
+        <sphere radius="0.1"/>
       </geometry>
     </visual>
@@ -46,5 +46,5 @@
       <origin xyz="-0.25 0 -0.1" rpy=" 0 0 0"/>
       <geometry>
-        <sphere radius="0.099"/>
+        <sphere radius="0.0998"/>
       </geometry>
     </collision>
@@ -52,9 +52,41 @@
       <origin xyz="-0.25 0 -0.1" rpy=" 0 0 0"/>
       <geometry>
-        <sphere radius="0.099"/>
+        <sphere radius="0.01"/>
       </geometry>
     </visual>
   </link>
 <!-- Add two wheels -->
+<link name='left_wheel'>
+   <pose>0 0 0.8 0 0 0</pose>
+    <inertial>
+      <mass value="5.0"/>
+      <origin xyz="0 0 0" rpy=" 0 0 0"/>
+      <inertia
+          ixx="0.1" ixy="0" ixz="0"
+          iyy="0.1" iyz="0"
+          izz="0.1"
+      />
+    </inertial>
+    <collision name='left_wheel_collision'>
+      <origin xyz="0 0 0" rpy=" 0 1.5707 1.5707"/>
+      <geometry>
+        <cylinder length="0.2" radius="0.05"/>
+      </geometry>
+    </collision>
+    <visual name='left_wheel_visual'>
+      <origin xyz="0 0 0" rpy=" 0 1.5707 1.5707"/>
+      <geometry>
+        <cylinder length="0.2" radius="0.05"/>
+      </geometry>
+    </visual>
+  </link>
+<joint type="continuous" name="left_wheel_hinge">
+	<origin xyz="0 0.3 0" rpy="0 0 0"/>
+	<child link="left_wheel"/>
+	<parent link="chassis"/>
+	<axis xyz="0 1 0" rpy="0 0 0"/>
+	<limit effort="10000" velocity="1000"/>
+	<dynamics damping="1.0" friction="1.0"/>
+</joint>
   <link name='right_wheel'>
    <pose>0 0 0.8 0 0 0</pose>
@@ -81,44 +113,12 @@
     </visual>
 </link>
-	<joint type="continuous" name="right_wheel_hinge">
-		<origin xyz="0 -0.3 0" rpy="0 0 0"/>
-		<child link="right_wheel"/>
-		<parent link="chassis"/>
-		<axis xyz="0 1 0" rpy="0 0 0"/>
-		<limit effort="10000" velocity="1000"/>
-		<dynamics damping="1.0" friction="1.0"/>
-	</joint>
-  <link name='left_wheel'>
-   <pose>0 0 0.8 0 0 0</pose>
-    <inertial>
-      <mass value="5.0"/>
-      <origin xyz="0 0 0" rpy=" 0 0 0"/>
-      <inertia
-          ixx="0.1" ixy="0" ixz="0"
-          iyy="0.1" iyz="0"
-          izz="0.1"
-      />
-    </inertial>
-    <collision name='left_wheel_collision'>
-      <origin xyz="0 0 0" rpy=" 0 1.5707 1.5707"/>
-      <geometry>
-        <cylinder length="0.2" radius="0.05"/>
-      </geometry>
-    </collision>
-    <visual name='left_wheel_visual'>
-      <origin xyz="0 0 0" rpy=" 0 1.5707 1.5707"/>
-      <geometry>
-        <cylinder length="0.2" radius="0.05"/>
-      </geometry>
-    </visual>
-  </link>
-	<joint type="continuous" name="left_wheel_hinge">
-		<origin xyz="0 0.3 0" rpy="0 0 0"/>
-		<child link="left_wheel"/>
-		<parent link="chassis"/>
-		<axis xyz="0 1 0" rpy="0 0 0"/>
-		<limit effort="10000" velocity="1000"/>
-		<dynamics damping="1.0" friction="1.0"/>
-	</joint>
+<joint type="continuous" name="right_wheel_hinge">
+	<origin xyz="0 -0.3 0" rpy="0 0 0"/>
+	<child link="right_wheel"/>
+	<parent link="chassis"/>
+	<axis xyz="0 1 0" rpy="0 0 0"/>
+	<limit effort="10000" velocity="1000"/>
+	<dynamics damping="1.0" friction="1.0"/>
+</joint>
   <!-- Add camera -->
   <link name='camera'>
@@ -178,9 +178,9 @@
     </visual>
   </link>
- <joint name="hokuyo_joint" type="fixed">
+  <joint type="fixed" name="hokuyo_joint">
+    <origin xyz="0.30 0 .1" rpy="0 0 0"/>
+    <child link="hokuyo"/>
+    <parent link="chassis"/>
     <axis xyz="0 1 0" rpy="0 0 0"/>
-    <origin xyz="0.15 0 0.1" rpy="0 0 0" />
-    <parent link="chassis"/>
-    <child link="hokuyo" />
   </joint>
 <gazebo reference="left_wheel">

Commit message: Update my_robot.xacro

File: my_robot/urdf/my_robot.xacro (robot description, xacro)
@@ -11,5 +11,5 @@
     <pose>0 0 0.1 0 0 0</pose>
     <inertial>
-      <mass value="30.0"/>
+      <mass value="15.0"/>
       <origin xyz="0.0 0 0" rpy=" 0 0 0"/>
       <inertia
@@ -22,5 +22,5 @@
       <origin xyz="0 0 0" rpy=" 0 0 0"/>
       <geometry>
-        <box size=".8 .4 .2"/>
+        <box size=".6 .3 .17"/>
       </geometry>
     </collision>
@@ -28,29 +28,29 @@
       <origin xyz="0 0 0" rpy=" 0 0 0"/>
       <geometry>
-        <box size=".8 .4 .2"/>
+        <box size=".6 .3 .17"/>
       </geometry>
     </visual>
     <collision name='back_caster_collision'>
-      <origin xyz="-0.25 0 -0.1" rpy=" 0 0 0"/>
+      <origin xyz="-0.225 0 -0.075" rpy=" 0 0 0"/>
       <geometry>
-        <sphere radius="0.0998"/>
+        <sphere radius="0.0749"/>
       </geometry>
     </collision>
     <visual name='back_caster_visual'>
-      <origin xyz="-0.25 0 -0.1" rpy=" 0 0 0"/>
+      <origin xyz="-0.225 0 -0.075" rpy=" 0 0 0"/>
       <geometry>
-        <sphere radius="0.1"/>
+        <sphere radius="0.075"/>
       </geometry>
     </visual>
     <collision name='front_caster_collision'>
-      <origin xyz="-0.25 0 -0.1" rpy=" 0 0 0"/>
+      <origin xyz="0.225 0 -0.075" rpy=" 0 0 0"/>
       <geometry>
-        <sphere radius="0.0998"/>
+        <sphere radius="0.0749"/>
       </geometry>
     </collision>
     <visual name='front_caster_visual'>
-      <origin xyz="-0.25 0 -0.1" rpy=" 0 0 0"/>
+      <origin xyz="0.225 0 -0.075" rpy=" 0 0 0"/>
       <geometry>
-        <sphere radius="0.01"/>
+        <sphere radius="0.075"/>
       </geometry>
     </visual>
@@ -58,8 +58,7 @@
 <!-- Add two wheels -->
 <link name='left_wheel'>
-   <pose>0 0 0.8 0 0 0</pose>
     <inertial>
       <mass value="5.0"/>
-      <origin xyz="0 0 0" rpy=" 0 0 0"/>
+      <origin xyz="0 0 0" rpy="0 1.5707 1.5707"/>
       <inertia
           ixx="0.1" ixy="0" ixz="0"
@@ -71,5 +70,5 @@
       <origin xyz="0 0 0" rpy=" 0 1.5707 1.5707"/>
       <geometry>
-        <cylinder length="0.2" radius="0.05"/>
+        <cylinder length="0.075" radius="0.15"/>
       </geometry>
     </collision>
@@ -77,10 +76,10 @@
       <origin xyz="0 0 0" rpy=" 0 1.5707 1.5707"/>
       <geometry>
-        <cylinder length="0.2" radius="0.05"/>
+        <cylinder length="0.075" radius="0.15"/>
       </geometry>
     </visual>
   </link>
 <joint type="continuous" name="left_wheel_hinge">
-	<origin xyz="0 0.3 0" rpy="0 0 0"/>
+	<origin xyz="0 0.25 0" rpy="0 0 0"/>
 	<child link="left_wheel"/>
 	<parent link="chassis"/>
@@ -90,8 +89,7 @@
 </joint>
   <link name='right_wheel'>
-   <pose>0 0 0.8 0 0 0</pose>
     <inertial>
       <mass value="5.0"/>
-      <origin xyz="0 0 0" rpy=" 0 0 0"/>
+      <origin xyz="0 0 0" rpy="0 1.5707 1.5707"/>
       <inertia
           ixx="0.1" ixy="0" ixz="0"
@@ -103,5 +101,5 @@
       <origin xyz="0 0 0" rpy=" 0 1.5707 1.5707"/>
       <geometry>
-        <cylinder length="0.2" radius="0.05"/>
+        <cylinder length="0.075" radius="0.15"/>
       </geometry>
     </collision>
@@ -109,10 +107,10 @@
       <origin xyz="0 0 0" rpy=" 0 1.5707 1.5707"/>
       <geometry>
-        <cylinder length="0.2" radius="0.05"/>
+        <cylinder length="0.075" radius="0.15"/>
       </geometry>
     </visual>
 </link>
 <joint type="continuous" name="right_wheel_hinge">
-	<origin xyz="0 -0.3 0" rpy="0 0 0"/>
+    	<origin xyz="0 -0.25 0" rpy="0 0 0"/>
 	<child link="right_wheel"/>
 	<parent link="chassis"/>
@@ -123,5 +121,4 @@
   <!-- Add camera -->
   <link name='camera'>
-    <pose>0 0 0 0 0 0</pose>
     <inertial>
       <mass value="0.1"/>
@@ -134,5 +131,5 @@
       />
     </inertial>
-    <collision name='collision'>
+    <collision name='camera_collision'>
       <origin xyz="0 0 0" rpy=" 0 0 0"/>
       <geometry>
@@ -148,5 +145,5 @@
   </link>
   <joint type="fixed" name="camera_joint">
-    <origin xyz="0.4 0 0" rpy="0 0 0"/>
+    <origin xyz="0.3 0 0" rpy="0 0 0"/>
     <child link="camera"/>
     <parent link="chassis"/>
@@ -155,5 +152,4 @@
   <!-- Add Lidar -->
   <link name='hokuyo'>
-    <pose>0 0 0 0 0 0</pose>
     <inertial>
       <mass value="1e-5"/>
@@ -165,5 +161,5 @@
       />
     </inertial>
-    <collision name='collision'>
+    <collision name='hokuyo_collision'>
       <origin xyz="0 0 0" rpy=" 0 0 0"/>
       <geometry>
@@ -179,5 +175,5 @@
   </link>
   <joint type="fixed" name="hokuyo_joint">
-    <origin xyz="0.30 0 .1" rpy="0 0 0"/>
+    <origin xyz="0.25 0 .15" rpy="0 0 0"/>
     <child link="hokuyo"/>
     <parent link="chassis"/>

Commit message: Update my_robot.xacro

File: my_robot/urdf/my_robot.xacro (robot description, xacro)
@@ -22,5 +22,5 @@
       <origin xyz="0 0 0" rpy=" 0 0 0"/>
       <geometry>
-        <box size=".6 .3 .17"/>
+        <box size=".6 .3 .15"/>
       </geometry>
     </collision>
@@ -28,5 +28,5 @@
       <origin xyz="0 0 0" rpy=" 0 0 0"/>
       <geometry>
-        <box size=".6 .3 .17"/>
+        <box size=".6 .3 .18"/>
       </geometry>
     </visual>

Commit message: Update my_robot.xacro

File: my_robot/urdf/my_robot.xacro (robot description, xacro)
@@ -22,5 +22,5 @@
       <origin xyz="0 0 0" rpy=" 0 0 0"/>
       <geometry>
-        <box size=".6 .3 .15"/>
+        <box size=".6 .3 .17"/>
       </geometry>
     </collision>
@@ -28,5 +28,5 @@
       <origin xyz="0 0 0" rpy=" 0 0 0"/>
       <geometry>
-        <box size=".6 .3 .18"/>
+        <box size=".6 .3 .17"/>
       </geometry>
     </visual>
